File: ESP32/PCB/EagleCAD/ESP32_EVKIT_v1.0.brd (EAGLE design)
At the start: 65 x 50 mm, 45 parts, among them IC1 AP7370Y, IC2 SN65HVD230, J1 O3, M1 ESP32_EVKIT_V1, SW1 ITS-1105-8, SW2 ITS-1105-8, X1 MICRO_SD_ATOM-A01482

Commit message: 메뉴얼 업로드
Parts:
- IC1: value AP7370Y -> AP7370Y-33Y
Changed lines of the file:
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@@
 <attribute name="VALUE" x="23.924" y="-5.399" size="0.7" layer="27" rot="R90"/>
 </element>
-<element name="IC1" library="cona_lib" package="SOT89" value="AP7370Y" x="23.325" y="6.8" smashed="yes" rot="R90">
+<element name="IC1" library="cona_lib" package="SOT89" value="AP7370Y-33Y" x="23.325" y="6.8" smashed="yes" rot="R90">
 <attribute name="NAME" x="19.95" y="6.035" size="0.7" layer="25" ratio="10" rot="R90"/>
 <attribute name="VALUE" x="27.6699" y="4.3949" size="0.7" layer="27" rot="R90"/>
