File: ESP32/PCB/EagleCAD/ESP32_EVKIT_v1.0.brd (EAGLE design)
At the start: 65 x 50 mm, 45 parts, among them IC1 AP7370Y-33Y, IC2 SN65HVD230, J1 O3, M1 ESP32_EVKIT_V1, SW1 ITS-1105-8, SW2 ITS-1105-8, X1 MICRO_SD_ATOM-A01482

Commit message: PCB TEST CODE UPDATE
Connections:
- net DAC1: now also JP1.2, M1.23; no longer C1.+, M1.22
- net DAC2: now also C1.+, M1.22; no longer JP1.2, M1.23
Routing:
- net DAC2: track 17.4 -> 12.3 mm
- net DAC1: track 12.3 -> 17.4 mm

Commit message: ARDUINO 예제 자료 업로드
Parts:
- R11: value 10k -> 1k
Changed lines of the file:
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@@
 <attribute name="VALUE" x="13.93" y="-6.26" size="0.7" layer="27" ratio="10" rot="R90"/>
 </element>
-<element name="R11" library="cona_lib" package="R0603" value="10k" x="43.2" y="15.525" smashed="yes">
+<element name="R11" library="cona_lib" package="R0603" value="1k" x="43.2" y="15.525" smashed="yes">
 <attribute name="NAME" x="41.624" y="15.809" size="0.7" layer="25" ratio="10" rot="R180"/>
 <attribute name="VALUE" x="41.676" y="14.001" size="0.7" layer="27" ratio="10"/>
