File: ESP32/PCB/EagleCAD/ESP32_EVKIT_v1.0.sch (EAGLE design)
At the start: 45 parts, among them IC1 AP7370Y, IC2 SN65HVD230, J1 O3, M1 ESP32_EVKIT_V1, SW1 ITS-1105-8, SW2 ITS-1105-8, X1 MICRO_SD_ATOM-A01482

Commit message: 메뉴얼 업로드
Parts:
- IC1: value AP7370Y -> AP7370Y-33Y
Changed lines of the file:
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@@
 <part name="PE38" library="cona_lib" deviceset="GND" device=""/>
 <part name="+3V16" library="cona_lib" deviceset="+3V3" device=""/>
-<part name="IC1" library="cona_lib" deviceset="AP7370" device="Y"/>
+<part name="IC1" library="cona_lib" deviceset="AP7370" device="Y" value="AP7370Y-33Y"/>
 <part name="PE17" library="cona_lib" deviceset="GND" device=""/>
 <part name="C2" library="cona_lib" deviceset="C_" device="0603" value="1uF"/>
@@
 <instance part="PAD1" gate="G$1" x="287.02" y="342.9" rot="R180"/>
 <instance part="R14" gate="G$1" x="281.94" y="322.58" rot="R90"/>
-<instance part="+3V1" gate="G$1" x="281.94" y="330.2"/>
+<instance part="+3V1" gate="G$1" x="281.94" y="332.74"/>
 <instance part="R13" gate="G$1" x="274.32" y="312.42" rot="R90"/>
 <instance part="+3V3" gate="G$1" x="274.32" y="325.12"/>
@@
 <pinref part="R14" gate="G$1" pin="2"/>
 <pinref part="+3V1" gate="G$1" pin="3V3"/>
-</segment>
-<segment>
+<wire x1="281.94" y1="330.2" x2="281.94" y2="327.66" width="0.1524" layer="91"/>
+</segment>
+<segment>

Commit message: PCB TEST CODE UPDATE
Connections:
- net DAC1: now also JP1.2, M1G$2.GPIO25; no longer C1.+, M1G$2.GPIO26
- net DAC2: now also C1.+, M1G$2.GPIO26; no longer JP1.2, M1G$2.GPIO25
Changed lines of the file:
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@@
-</segment>
-</net>
-<net name="DAC2" class="0">
-<segment>
-<pinref part="M1" gate="G$2" pin="GPIO25"/>
-<wire x1="243.84" y1="340.36" x2="261.62" y2="340.36" width="0.1524" layer="91"/>
-<label x="246.38" y="340.36" size="1.778" layer="95"/>
-</segment>
-<segment>
-<pinref part="JP1" gate="G$1" pin="2"/>
-<wire x1="104.14" y1="388.62" x2="91.44" y2="388.62" width="0.1524" layer="91"/>
-<label x="93.98" y="388.62" size="1.778" layer="95"/>
-</segment>
-</net>
-<net name="DAC1" class="0">
-<segment>
-<pinref part="M1" gate="G$2" pin="GPIO26"/>
-<wire x1="243.84" y1="342.9" x2="261.62" y2="342.9" width="0.1524" layer="91"/>
-<label x="246.38" y="342.9" size="1.778" layer="95"/>
-</segment>
-<segment>
-<pinref part="C1" gate="G$1" pin="+"/>
-<wire x1="93.98" y1="393.7" x2="83.82" y2="393.7" width="0.1524" layer="91"/>
-<label x="86.36" y="393.7" size="1.778" layer="95"/>
 </segment>
 </net>
@@
 </segment>
 </net>
+<net name="DAC1" class="0">
+<segment>
+<pinref part="M1" gate="G$2" pin="GPIO25"/>
+<wire x1="243.84" y1="340.36" x2="261.62" y2="340.36" width="0.1524" layer="91"/>
+<label x="246.38" y="340.36" size="1.778" layer="95"/>
+</segment>
+<segment>
+<pinref part="JP1" gate="G$1" pin="2"/>
+<wire x1="104.14" y1="388.62" x2="91.44" y2="388.62" width="0.1524" layer="91"/>
+<label x="93.98" y="388.62" size="1.778" layer="95"/>
+</segment>
+</net>
+<net name="DAC2" class="0">
+<segment>
+<pinref part="C1" gate="G$1" pin="+"/>
+<wire x1="93.98" y1="393.7" x2="83.82" y2="393.7" width="0.1524" layer="91"/>
+<label x="86.36" y="393.7" size="1.778" layer="95"/>
+</segment>
+<segment>
+<pinref part="M1" gate="G$2" pin="GPIO26"/>
+<wire x1="243.84" y1="342.9" x2="261.62" y2="342.9" width="0.1524" layer="91"/>
+<label x="246.38" y="342.9" size="1.778" layer="95"/>
+</segment>
+</net>

Commit message: ARDUINO 예제 자료 업로드
Parts:
- R11: value 10k -> 1k
Changed lines of the file:
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@@
 <part name="PE22" library="cona_lib" deviceset="GND" device=""/>
 <part name="X1" library="cona_lib" deviceset="MICRO_SD_ATOM-A01482" device=""/>
-<part name="R11" library="cona_lib" deviceset="R_" device="0603" value="10k"/>
+<part name="R11" library="cona_lib" deviceset="R_" device="0603" value="1k"/>
 <part name="JP6" library="cona_lib" deviceset="MA02" device="ED350V-02P" value="ED350V-02P"/>
 <part name="C1" library="cona_lib" deviceset="CP_" device="2012" value="10uF"/>
